Commit message: feat: cập nhật thông số kích thước xe thực tế
- base: 304×268×84 mm
- wheel_radius: 100 mm, wheel_width: 29 mm
- wheelbase: 210 mm, track_width: 217 mm
- nav2 robot_radius: 0.21 m (circumscribed)
- Cập nhật inertia URDF theo kích thước mới

Co-Authored-By: Claude Sonnet 4.6 <noreply@anthropic.com>

File: src/amr_description/urdf/amr.urdf.xacro (robot description, xacro)
@@ -8,11 +8,11 @@
   <!-- ─── Tham số kích thước (đơn vị: mét) ─────────────────────── -->
   <!-- CẦN ĐIỀU CHỈNH theo kích thước khung xe thực tế -->
-  <xacro:property name="base_length"   value="0.30"/>  <!-- chiều dài -->
-  <xacro:property name="base_width"    value="0.20"/>  <!-- chiều rộng -->
-  <xacro:property name="base_height"   value="0.08"/>  <!-- chiều cao chassis -->
-  <xacro:property name="wheel_radius"  value="0.04"/>  <!-- bán kính bánh -->
-  <xacro:property name="wheel_width"   value="0.025"/> <!-- bề rộng bánh -->
-  <xacro:property name="wheelbase"     value="0.22"/>  <!-- khoảng cách trục trước-sau -->
-  <xacro:property name="track_width"   value="0.18"/>  <!-- khoảng cách 2 bánh ngang -->
+  <xacro:property name="base_length"   value="0.304"/> <!-- chiều dài -->
+  <xacro:property name="base_width"    value="0.268"/> <!-- chiều rộng -->
+  <xacro:property name="base_height"   value="0.084"/> <!-- chiều cao chassis -->
+  <xacro:property name="wheel_radius"  value="0.10"/>  <!-- bán kính bánh -->
+  <xacro:property name="wheel_width"   value="0.029"/> <!-- bề rộng bánh -->
+  <xacro:property name="wheelbase"     value="0.21"/>  <!-- khoảng cách trục trước-sau -->
+  <xacro:property name="track_width"   value="0.217"/> <!-- khoảng cách 2 bánh ngang -->
   <!-- ─── Materials ─────────────────────────────────────────────── -->
   <material name="dark_grey">
@@ -50,8 +50,8 @@
     <inertial>
       <mass value="2.0"/>
-      <!-- Điều chỉnh inertia theo khối lượng thực tế -->
-      <inertia ixx="0.012" ixy="0" ixz="0"
-               iyy="0.020" iyz="0"
-               izz="0.028"/>
+      <!-- Inertia tính cho hộp đặc m=2kg, L=0.304 W=0.268 H=0.084 -->
+      <inertia ixx="0.0132" ixy="0" ixz="0"
+               iyy="0.0166" iyz="0"
+               izz="0.0274"/>
     </inertial>
   </link>

Commit message: fix: correct wheel inertia values for simulation
Co-Authored-By: Claude Opus 4.8 <noreply@anthropic.com>

File: src/amr_description/urdf/amr.urdf.xacro (robot description, xacro)
@@ -74,7 +74,7 @@
       <inertial>
         <mass value="0.15"/>
-        <inertia ixx="0.0002" ixy="0" ixz="0"
-                 iyy="0.0002" iyz="0"
-                 izz="0.0003"/>
+        <inertia ixx="0.0004" ixy="0.0" ixz="0.0"
+                 iyy="0.0004" iyz="0.0"
+                 izz="0.00075"/>
       </inertial>
     </link>

Commit message: fix: correct wheel radius 100mm->50mm and wheel lateral position
Co-Authored-By: Claude Opus 4.8 <noreply@anthropic.com>

File: src/amr_description/urdf/amr.urdf.xacro (robot description, xacro)
@@ -11,8 +11,8 @@
   <xacro:property name="base_width"    value="0.268"/> <!-- chiều rộng -->
   <xacro:property name="base_height"   value="0.084"/> <!-- chiều cao chassis -->
-  <xacro:property name="wheel_radius"  value="0.10"/>  <!-- bán kính bánh -->
+  <xacro:property name="wheel_radius"  value="0.05"/>  <!-- bán kính bánh (đường kính 100mm → r=50mm) -->
   <xacro:property name="wheel_width"   value="0.029"/> <!-- bề rộng bánh -->
   <xacro:property name="wheelbase"     value="0.21"/>  <!-- khoảng cách trục trước-sau -->
-  <xacro:property name="track_width"   value="0.217"/> <!-- khoảng cách 2 bánh ngang -->
+  <xacro:property name="track_width"   value="0.333"/> <!-- khoảng cách 2 tâm bánh ngang: 2×(134 + 18 + wheel_width/2) = 2×166.5mm -->
   <!-- ─── Materials ─────────────────────────────────────────────── -->
   <material name="dark_grey">

Commit message: fix: set track_width 0.217m, frame width 0.158m, add wheel_inner_gap
Co-Authored-By: Claude Opus 4.8 <noreply@anthropic.com>

File: src/amr_description/urdf/amr.urdf.xacro (robot description, xacro)
@@ -9,10 +9,12 @@
   <!-- CẦN ĐIỀU CHỈNH theo kích thước khung xe thực tế -->
   <xacro:property name="base_length"   value="0.304"/> <!-- chiều dài -->
-  <xacro:property name="base_width"    value="0.268"/> <!-- chiều rộng -->
+  <xacro:property name="base_width"    value="0.158"/> <!-- chiều rộng khung chassis thật (không gồm bánh) -->
   <xacro:property name="base_height"   value="0.084"/> <!-- chiều cao chassis -->
   <xacro:property name="wheel_radius"  value="0.05"/>  <!-- bán kính bánh (đường kính 100mm → r=50mm) -->
   <xacro:property name="wheel_width"   value="0.029"/> <!-- bề rộng bánh -->
   <xacro:property name="wheelbase"     value="0.21"/>  <!-- khoảng cách trục trước-sau -->
-  <xacro:property name="track_width"   value="0.333"/> <!-- khoảng cách 2 tâm bánh ngang: 2×(134 + 18 + wheel_width/2) = 2×166.5mm -->
+  <xacro:property name="track_width"   value="0.217"/> <!-- khoảng cách 2 tâm bánh ngang (tâm→tâm) -->
+  <!-- Khoảng trống lọt lòng giữa 2 mặt trong của 2 bánh (dẫn xuất) = 0.188m -->
+  <xacro:property name="wheel_inner_gap" value="${track_width - wheel_width}"/>
   <!-- ─── Materials ─────────────────────────────────────────────── -->
   <material name="dark_grey">

Commit message: fix: recompute base_link and wheel inertia for new dimensions
Co-Authored-By: Claude Opus 4.8 <noreply@anthropic.com>

File: src/amr_description/urdf/amr.urdf.xacro (robot description, xacro)
@@ -52,8 +52,8 @@
     <inertial>
       <mass value="2.0"/>
-      <!-- Inertia tính cho hộp đặc m=2kg, L=0.304 W=0.268 H=0.084 -->
-      <inertia ixx="0.0132" ixy="0" ixz="0"
-               iyy="0.0166" iyz="0"
-               izz="0.0274"/>
+      <!-- Hộp đặc m=2kg, L=0.304 W=0.158 H=0.084: I=1/12·m·(a²+b²) -->
+      <inertia ixx="0.005337" ixy="0" ixz="0"
+               iyy="0.016579" iyz="0"
+               izz="0.019563"/>
     </inertial>
   </link>
@@ -76,7 +76,8 @@
       <inertial>
         <mass value="0.15"/>
-        <inertia ixx="0.0004" ixy="0.0" ixz="0.0"
-                 iyy="0.0004" iyz="0.0"
-                 izz="0.00075"/>
+        <!-- Trụ đặc r=0.05 h=0.029, trục quay Y: iyy=½mr², ixx=izz=1/12·m·(3r²+h²) -->
+        <inertia ixx="0.0001043" ixy="0.0" ixz="0.0"
+                 iyy="0.0001875" iyz="0.0"
+                 izz="0.0001043"/>
       </inertial>
     </link>

Commit message: fix: update chassis dimensions L=297mm H=62mm ground_clearance=22mm
Co-Authored-By: Claude Opus 4.8 <noreply@anthropic.com>

File: src/amr_description/urdf/amr.urdf.xacro (robot description, xacro)
@@ -8,7 +8,8 @@
   <!-- ─── Tham số kích thước (đơn vị: mét) ─────────────────────── -->
   <!-- CẦN ĐIỀU CHỈNH theo kích thước khung xe thực tế -->
-  <xacro:property name="base_length"   value="0.304"/> <!-- chiều dài -->
+  <xacro:property name="base_length"   value="0.297"/> <!-- chiều dài chassis (không tính bánh) -->
   <xacro:property name="base_width"    value="0.158"/> <!-- chiều rộng khung chassis thật (không gồm bánh) -->
-  <xacro:property name="base_height"   value="0.084"/> <!-- chiều cao chassis -->
+  <xacro:property name="base_height"   value="0.062"/> <!-- chiều cao chassis (không tính bánh) -->
+  <xacro:property name="ground_clearance" value="0.022"/> <!-- mặt đất → mặt dưới khung gầm -->
   <xacro:property name="wheel_radius"  value="0.05"/>  <!-- bán kính bánh (đường kính 100mm → r=50mm) -->
   <xacro:property name="wheel_width"   value="0.029"/> <!-- bề rộng bánh -->
@@ -17,4 +18,6 @@
   <!-- Khoảng trống lọt lòng giữa 2 mặt trong của 2 bánh (dẫn xuất) = 0.188m -->
   <xacro:property name="wheel_inner_gap" value="${track_width - wheel_width}"/>
+  <!-- z của base_link so với base_footprint = ground_clearance + chassis_height/2 = 0.053m -->
+  <xacro:property name="base_link_z" value="${ground_clearance + base_height/2}"/>
   <!-- ─── Materials ─────────────────────────────────────────────── -->
   <material name="dark_grey">
@@ -35,5 +38,5 @@
     <parent link="base_footprint"/>
     <child  link="base_link"/>
-    <origin xyz="0 0 ${wheel_radius}" rpy="0 0 0"/>
+    <origin xyz="0 0 ${base_link_z}" rpy="0 0 0"/>
   </joint>
   <!-- ─── Base link (chassis) ───────────────────────────────────── -->
@@ -52,8 +55,8 @@
     <inertial>
       <mass value="2.0"/>
-      <!-- Hộp đặc m=2kg, L=0.304 W=0.158 H=0.084: I=1/12·m·(a²+b²) -->
-      <inertia ixx="0.005337" ixy="0" ixz="0"
-               iyy="0.016579" iyz="0"
-               izz="0.019563"/>
+      <!-- Hộp đặc m=2kg, L=0.297 W=0.158 H=0.062: I=1/12·m·(a²+b²) -->
+      <inertia ixx="0.004801" ixy="0" ixz="0"
+               iyy="0.015342" iyz="0"
+               izz="0.018862"/>
     </inertial>
   </link>
@@ -85,5 +88,6 @@
       <parent link="base_link"/>
       <child  link="${name}_wheel"/>
-      <origin xyz="${x} ${y} 0" rpy="0 0 0"/>
+      <!-- z = wheel_radius - base_link_z = 0.05 - 0.053 = -0.003m (tâm bánh hơi thấp hơn tâm chassis) -->
+      <origin xyz="${x} ${y} ${wheel_radius - base_link_z}" rpy="0 0 0"/>
       <axis xyz="0 1 0"/>
     </joint>

Commit message: refactor(amr_description): tách amr.urdf.xacro thành cấu trúc modular
- inertial_macros.xacro: macro inertial_box và inertial_cylinder (thay thế giá trị hardcode)
- amr_core.xacro: properties, materials, base_link, wheel macro + 4 bánh
- lidar.xacro: laser_frame + laser_joint
- camera.xacro: camera_frame, camera_optical_frame và các joint
- ros2_control.xacro: skeleton trống cho giai đoạn Nav2
- amr.urdf.xacro: chỉ còn <robot> root + 5 xacro:include

Co-Authored-By: Claude Sonnet 4.6 <noreply@anthropic.com>

File: src/amr_description/urdf/amr.urdf.xacro (robot description, xacro)
@@ -4,141 +4,9 @@
        AMR Ackermann Robot — URDF/Xacro
        Hardware: Jetson Orin Nano + STM32F446RE
-       Điều chỉnh kích thước theo khung xe thực tế
   ═══════════════════════════════════════════════════════════════ -->
-  <!-- ─── Tham số kích thước (đơn vị: mét) ─────────────────────── -->
-  <!-- CẦN ĐIỀU CHỈNH theo kích thước khung xe thực tế -->
-  <xacro:property name="base_length"   value="0.297"/> <!-- chiều dài chassis (không tính bánh) -->
-  <xacro:property name="base_width"    value="0.158"/> <!-- chiều rộng khung chassis thật (không gồm bánh) -->
-  <xacro:property name="base_height"   value="0.062"/> <!-- chiều cao chassis (không tính bánh) -->
-  <xacro:property name="ground_clearance" value="0.022"/> <!-- mặt đất → mặt dưới khung gầm -->
-  <xacro:property name="wheel_radius"  value="0.05"/>  <!-- bán kính bánh (đường kính 100mm → r=50mm) -->
-  <xacro:property name="wheel_width"   value="0.029"/> <!-- bề rộng bánh -->
-  <xacro:property name="wheelbase"     value="0.21"/>  <!-- khoảng cách trục trước-sau -->
-  <xacro:property name="track_width"   value="0.217"/> <!-- khoảng cách 2 tâm bánh ngang (tâm→tâm) -->
-  <!-- Khoảng trống lọt lòng giữa 2 mặt trong của 2 bánh (dẫn xuất) = 0.188m -->
-  <xacro:property name="wheel_inner_gap" value="${track_width - wheel_width}"/>
-  <!-- z của base_link so với base_footprint = ground_clearance + chassis_height/2 = 0.053m -->
-  <xacro:property name="base_link_z" value="${ground_clearance + base_height/2}"/>
-  <!-- ─── Materials ─────────────────────────────────────────────── -->
-  <material name="dark_grey">
-    <color rgba="0.2 0.2 0.2 1.0"/>
-  </material>
-  <material name="light_grey">
-    <color rgba="0.7 0.7 0.7 1.0"/>
-  </material>
-  <material name="blue">
-    <color rgba="0.0 0.4 0.8 1.0"/>
-  </material>
-  <material name="black">
-    <color rgba="0.1 0.1 0.1 1.0"/>
-  </material>
-  <!-- ─── Base footprint ────────────────────────────────────────── -->
-  <link name="base_footprint"/>
-  <joint name="base_footprint_joint" type="fixed">
-    <parent link="base_footprint"/>
-    <child  link="base_link"/>
-    <origin xyz="0 0 ${base_link_z}" rpy="0 0 0"/>
-  </joint>
-  <!-- ─── Base link (chassis) ───────────────────────────────────── -->
-  <link name="base_link">
-    <visual>
-      <geometry>
-        <box size="${base_length} ${base_width} ${base_height}"/>
-      </geometry>
-      <material name="dark_grey"/>
-    </visual>
-    <collision>
-      <geometry>
-        <box size="${base_length} ${base_width} ${base_height}"/>
-      </geometry>
-    </collision>
-    <inertial>
-      <mass value="2.0"/>
-      <!-- Hộp đặc m=2kg, L=0.297 W=0.158 H=0.062: I=1/12·m·(a²+b²) -->
-      <inertia ixx="0.004801" ixy="0" ixz="0"
-               iyy="0.015342" iyz="0"
-               izz="0.018862"/>
-    </inertial>
-  </link>
-  <!-- ─── Wheel macro ───────────────────────────────────────────── -->
-  <xacro:macro name="wheel" params="name x y mirrored">
-    <link name="${name}_wheel">
-      <visual>
-        <geometry>
-          <cylinder radius="${wheel_radius}" length="${wheel_width}"/>
-        </geometry>
-        <origin xyz="0 0 0" rpy="${pi/2} 0 0"/>
-        <material name="black"/>
-      </visual>
-      <collision>
-        <geometry>
-          <cylinder radius="${wheel_radius}" length="${wheel_width}"/>
-        </geometry>
-        <origin xyz="0 0 0" rpy="${pi/2} 0 0"/>
-      </collision>
-      <inertial>
-        <mass value="0.15"/>
-        <!-- Trụ đặc r=0.05 h=0.029, trục quay Y: iyy=½mr², ixx=izz=1/12·m·(3r²+h²) -->
-        <inertia ixx="0.0001043" ixy="0.0" ixz="0.0"
-                 iyy="0.0001875" iyz="0.0"
-                 izz="0.0001043"/>
-      </inertial>
-    </link>
-    <joint name="${name}_wheel_joint" type="continuous">
-      <parent link="base_link"/>
-      <child  link="${name}_wheel"/>
-      <!-- z = wheel_radius - base_link_z = 0.05 - 0.053 = -0.003m (tâm bánh hơi thấp hơn tâm chassis) -->
-      <origin xyz="${x} ${y} ${wheel_radius - base_link_z}" rpy="0 0 0"/>
-      <axis xyz="0 1 0"/>
-    </joint>
-  </xacro:macro>
-  <!-- Bánh sau dẫn động (JGB37-520) -->
-  <xacro:wheel name="rear_left"
-    x="${-wheelbase/2}" y="${track_width/2}"  mirrored="0"/>
-  <xacro:wheel name="rear_right"
-    x="${-wheelbase/2}" y="${-track_width/2}" mirrored="1"/>
-  <!-- Bánh trước lái (HTS-20H) — dùng fixed joint, servo tính riêng -->
-  <xacro:wheel name="front_left"
-    x="${wheelbase/2}"  y="${track_width/2}"  mirrored="0"/>
-  <xacro:wheel name="front_right"
-    x="${wheelbase/2}"  y="${-track_width/2}" mirrored="1"/>
-  <!-- ─── LiDAR frame ───────────────────────────────────────────── -->
-  <!-- CẦN ĐIỀU CHỈNH vị trí gắn LiDAR trên xe thực tế -->
-  <link name="laser_frame">
-    <visual>
-      <geometry>
-        <cylinder radius="0.035" length="0.06"/>
-      </geometry>
-      <material name="blue"/>
-    </visual>
-  </link>
-  <joint name="laser_joint" type="fixed">
-    <parent link="base_link"/>
-    <child  link="laser_frame"/>
-    <!-- Điều chỉnh xyz theo vị trí thực tế của RPLidar trên xe -->
-    <origin xyz="0.10 0 0.06" rpy="0 0 0"/>
-  </joint>
-  <!-- ─── Camera frame ──────────────────────────────────────────── -->
-  <!-- CẦN ĐIỀU CHỈNH vị trí gắn camera IMX-219 -->
-  <link name="camera_frame">
-    <visual>
-      <geometry>
-        <box size="0.025 0.025 0.020"/>
-      </geometry>
-      <material name="light_grey"/>
-    </visual>
-  </link>
-  <joint name="camera_joint" type="fixed">
-    <parent link="base_link"/>
-    <child  link="camera_frame"/>
-    <!-- Điều chỉnh xyz: camera thường gắn phía trước, hướng xuống hoặc thẳng -->
-    <origin xyz="0.12 0 0.05" rpy="0 0.3 0"/>
-  </joint>
-  <!-- Frame optical của camera (ROS convention: z-forward, x-right, y-down) -->
-  <link name="camera_optical_frame"/>
-  <joint name="camera_optical_joint" type="fixed">
-    <parent link="camera_frame"/>
-    <child  link="camera_optical_frame"/>
-    <origin xyz="0 0 0" rpy="${-pi/2} 0 ${-pi/2}"/>
-  </joint>
+  <xacro:include filename="$(find amr_description)/urdf/inertial_macros.xacro"/>
+  <xacro:include filename="$(find amr_description)/urdf/amr_core.xacro"/>
+  <xacro:include filename="$(find amr_description)/urdf/lidar.xacro"/>
+  <xacro:include filename="$(find amr_description)/urdf/camera.xacro"/>
+  <xacro:include filename="$(find amr_description)/urdf/ros2_control.xacro"/>
 </robot>
