Commit message: feat(amr_description): thêm Gazebo Fortress simulation support
URDF:
- amr_core.xacro: tách steering_wheel macro riêng (front_left/right_steer_joint
  revolute ±30°), thêm <gazebo> friction mu1=1.0/mu2=0.5 cho 4 bánh, màu links
- ros2_control.xacro: IgnitionSystem plugin với velocity cmd bánh sau,
  position cmd steer joints, passive state-only cho bánh trước

Config:
- config/controller_gz_sim.yaml: AckermannSteeringController + JointStateBroadcaster
  (wheelbase=0.21m, track=0.217m, r=0.05m)
- config/gz_bridge.yaml: bridge /cmd_vel /odom /scan /clock /joint_states /tf

Launch:
- launch/gazebo.launch.py: robot_state_publisher → ign gazebo → spawn
  → controllers (jsb trước, ackermann sau) → ros_gz_bridge (delay 3s)

CMakeLists.txt: thêm config/ vào install directories

Co-Authored-By: Claude Sonnet 4.6 <noreply@anthropic.com>

File: src/amr_description/urdf/amr_core.xacro (robot description, xacro)
@@ -50,6 +50,6 @@
     <xacro:inertial_box mass="2.0" l="${base_length}" w="${base_width}" h="${base_height}"/>
   </link>
-  <!-- ─── Wheel macro ───────────────────────────────────────────── -->
-  <xacro:macro name="wheel" params="name x y mirrored">
+  <!-- ─── Wheel macro (bánh sau dẫn động) ─────────────────────── -->
+  <xacro:macro name="wheel" params="name x y">
     <link name="${name}_wheel">
       <visual>
@@ -71,14 +71,87 @@
       <parent link="base_link"/>
       <child  link="${name}_wheel"/>
-      <!-- z = wheel_radius - base_link_z = 0.05 - 0.053 = -0.003m (tâm bánh hơi thấp hơn tâm chassis) -->
+      <!-- z = wheel_radius - base_link_z = 0.05 - 0.053 = -0.003m -->
       <origin xyz="${x} ${y} ${wheel_radius - base_link_z}" rpy="0 0 0"/>
       <axis xyz="0 1 0"/>
     </joint>
   </xacro:macro>
+  <!-- ─── Steering wheel macro (bánh trước lái) ────────────────── -->
+  <!-- Cấu trúc: base_link → steer_joint (revolute,z) → steer_link
+                            → wheel_joint (continuous,y) → wheel    -->
+  <xacro:macro name="steering_wheel" params="name x y">
+    <!-- Link trung gian tại tâm bánh, chỉ mang inertia tối thiểu -->
+    <link name="${name}_steer_link">
+      <xacro:inertial_box mass="0.001" l="0.01" w="0.01" h="0.01"/>
+    </link>
+    <!-- Joint lái: revolute quanh trục Z, giới hạn ±30° -->
+    <joint name="${name}_steer_joint" type="revolute">
+      <parent link="base_link"/>
+      <child  link="${name}_steer_link"/>
+      <origin xyz="${x} ${y} ${wheel_radius - base_link_z}" rpy="0 0 0"/>
+      <axis xyz="0 0 1"/>
+      <limit lower="-0.5236" upper="0.5236" effort="10.0" velocity="1.0"/>
+      <dynamics damping="0.1" friction="0.1"/>
+    </joint>
+    <!-- Bánh trước: xoay quanh Y, parent là steer_link -->
+    <link name="${name}_wheel">
+      <visual>
+        <geometry>
+          <cylinder radius="${wheel_radius}" length="${wheel_width}"/>
+        </geometry>
+        <origin xyz="0 0 0" rpy="${pi/2} 0 0"/>
+        <material name="black"/>
+      </visual>
+      <collision>
+        <geometry>
+          <cylinder radius="${wheel_radius}" length="${wheel_width}"/>
+        </geometry>
+        <origin xyz="0 0 0" rpy="${pi/2} 0 0"/>
+      </collision>
+      <xacro:inertial_cylinder mass="0.15" r="${wheel_radius}" h="${wheel_width}"/>
+    </link>
+    <joint name="${name}_wheel_joint" type="continuous">
+      <parent link="${name}_steer_link"/>
+      <child  link="${name}_wheel"/>
+      <origin xyz="0 0 0" rpy="0 0 0"/>
+      <axis xyz="0 1 0"/>
+    </joint>
+  </xacro:macro>
   <!-- Bánh sau dẫn động (JGB37-520) -->
-  <xacro:wheel name="rear_left"   x="${-wheelbase/2}" y="${track_width/2}"  mirrored="0"/>
-  <xacro:wheel name="rear_right"  x="${-wheelbase/2}" y="${-track_width/2}" mirrored="1"/>
-  <!-- Bánh trước lái (HTS-20H) — dùng fixed joint, servo tính riêng -->
-  <xacro:wheel name="front_left"  x="${wheelbase/2}"  y="${track_width/2}"  mirrored="0"/>
-  <xacro:wheel name="front_right" x="${wheelbase/2}"  y="${-track_width/2}" mirrored="1"/>
+  <xacro:wheel name="rear_left"   x="${-wheelbase/2}" y="${track_width/2}"/>
+  <xacro:wheel name="rear_right"  x="${-wheelbase/2}" y="${-track_width/2}"/>
+  <!-- Bánh trước lái (HTS-20H) — có revolute steer_joint cho Ackermann controller -->
+  <xacro:steering_wheel name="front_left"  x="${wheelbase/2}"  y="${track_width/2}"/>
+  <xacro:steering_wheel name="front_right" x="${wheelbase/2}"  y="${-track_width/2}"/>
+  <!-- ─── Gazebo: friction cho bánh ────────────────────────────── -->
+  <!-- mu1 = hệ số ma sát tĩnh, mu2 = hệ số ma sát trượt -->
+  <gazebo reference="rear_left_wheel">
+    <mu1>1.0</mu1>
+    <mu2>0.5</mu2>
+    <material>Gazebo/Black</material>
+  </gazebo>
+  <gazebo reference="rear_right_wheel">
+    <mu1>1.0</mu1>
+    <mu2>0.5</mu2>
+    <material>Gazebo/Black</material>
+  </gazebo>
+  <gazebo reference="front_left_wheel">
+    <mu1>1.0</mu1>
+    <mu2>0.5</mu2>
+    <material>Gazebo/Black</material>
+  </gazebo>
+  <gazebo reference="front_right_wheel">
+    <mu1>1.0</mu1>
+    <mu2>0.5</mu2>
+    <material>Gazebo/Black</material>
+  </gazebo>
+  <!-- ─── Gazebo: màu sắc các link ──────────────────────────────── -->
+  <gazebo reference="base_link">
+    <material>Gazebo/DarkGrey</material>
+  </gazebo>
+  <gazebo reference="front_left_steer_link">
+    <material>Gazebo/Grey</material>
+  </gazebo>
+  <gazebo reference="front_right_steer_link">
+    <material>Gazebo/Grey</material>
+  </gazebo>
 </robot>

File: src/amr_description/urdf/ros2_control.xacro (robot description, xacro)
@@ -1,6 +1,62 @@
 <?xml version="1.0"?>
 <robot xmlns:xacro="http://www.ros.org/wiki/xacro">
-  <!-- ─── ros2_control hardware interface ──────────────────────── -->
-  <!-- TODO Giai đoạn 5: khai báo <ros2_control> hardware interface -->
-  <!-- Tham khảo: https://control.ros.org/humble/               -->
+  <!-- ─── ros2_control — Ignition Fortress hardware interface ─────── -->
+  <ros2_control name="IgnitionSystem" type="system">
+    <hardware>
+      <!-- Plugin cho Gazebo Fortress (Ignition) -->
+      <plugin>ign_ros2_control/IgnitionSystem</plugin>
+    </hardware>
+    <!-- Bánh sau trái — velocity command (dẫn động) -->
+    <joint name="rear_left_wheel_joint">
+      <command_interface name="velocity">
+        <param name="min">-10</param>
+        <param name="max">10</param>
+      </command_interface>
+      <state_interface name="position"/>
+      <state_interface name="velocity"/>
+    </joint>
+    <!-- Bánh sau phải — velocity command (dẫn động) -->
+    <joint name="rear_right_wheel_joint">
+      <command_interface name="velocity">
+        <param name="min">-10</param>
+        <param name="max">10</param>
+      </command_interface>
+      <state_interface name="position"/>
+      <state_interface name="velocity"/>
+    </joint>
+    <!-- Khớp lái trước trái — position command -->
+    <joint name="front_left_steer_joint">
+      <command_interface name="position">
+        <param name="min">-0.5236</param>
+        <param name="max">0.5236</param>
+      </command_interface>
+      <state_interface name="position"/>
+      <state_interface name="velocity"/>
+    </joint>
+    <!-- Khớp lái trước phải — position command -->
+    <joint name="front_right_steer_joint">
+      <command_interface name="position">
+        <param name="min">-0.5236</param>
+        <param name="max">0.5236</param>
+      </command_interface>
+      <state_interface name="position"/>
+      <state_interface name="velocity"/>
+    </joint>
+    <!-- Bánh trước — passive (không command, chỉ đọc state) -->
+    <joint name="front_left_wheel_joint">
+      <state_interface name="position"/>
+      <state_interface name="velocity"/>
+    </joint>
+    <joint name="front_right_wheel_joint">
+      <state_interface name="position"/>
+      <state_interface name="velocity"/>
+    </joint>
+  </ros2_control>
+  <!-- Plugin ign_ros2_control tải vào Gazebo Fortress -->
+  <gazebo>
+    <plugin filename="ign_ros2_control-system"
+            name="ign_ros2_control::IgnRos2ControlPlugin">
+      <parameters>$(find amr_description)/config/controller_gz_sim.yaml</parameters>
+    </plugin>
+  </gazebo>
 </robot>

Commit message: feat(amr_description): merge quy ước trục Z bánh xe + steering joints từ repo bạn bè
- amr_core.xacro: đổi trục quay bánh xe Y -> Z (frame xoay -90° quanh X
  qua origin của joint), thêm param mirrored cho bánh đối xứng
- steer_link đặt tại mặt phẳng base_link (z=0), kingpin lái axis Z
- giữ nguyên tên links/joints, wheelbase=0.21, track=0.217, kích thước
- controller_gz_sim.yaml: sửa tên param theo steering_controllers_library
  (traction_joints_names/steering_joints_names/traction_track_width/...)
  khớp version controller đã cài -> fix lỗi "string_array got [not set]"

Co-Authored-By: Claude Opus 4.8 <noreply@anthropic.com>

File: src/amr_description/urdf/amr_core.xacro (robot description, xacro)
@@ -51,5 +51,9 @@
   </link>
   <!-- ─── Wheel macro (bánh sau dẫn động) ─────────────────────── -->
-  <xacro:macro name="wheel" params="name x y">
+  <!-- Quy ước trục Z (theo repo bạn bè): cả frame của bánh được xoay  -->
+  <!-- -90° quanh X qua origin của joint, nên trục quay khai báo là Z  -->
+  <!-- (0 0 1) trong frame đã xoay → ứng với trục Y thế giới (lăn tới). -->
+  <!-- mirrored=1 → +90° thay vì -90° (lật chiều trục cho bánh đối xứng).-->
+  <xacro:macro name="wheel" params="name y mirrored">
     <link name="${name}_wheel">
       <visual>
@@ -57,5 +61,4 @@
           <cylinder radius="${wheel_radius}" length="${wheel_width}"/>
         </geometry>
-        <origin xyz="0 0 0" rpy="${pi/2} 0 0"/>
         <material name="black"/>
       </visual>
@@ -64,5 +67,4 @@
           <cylinder radius="${wheel_radius}" length="${wheel_width}"/>
         </geometry>
-        <origin xyz="0 0 0" rpy="${pi/2} 0 0"/>
       </collision>
       <xacro:inertial_cylinder mass="0.15" r="${wheel_radius}" h="${wheel_width}"/>
@@ -72,13 +74,17 @@
       <child  link="${name}_wheel"/>
       <!-- z = wheel_radius - base_link_z = 0.05 - 0.053 = -0.003m -->
-      <origin xyz="${x} ${y} ${wheel_radius - base_link_z}" rpy="0 0 0"/>
-      <axis xyz="0 1 0"/>
+      <origin xyz="${-wheelbase/2} ${y} ${wheel_radius - base_link_z}"
+              rpy="${-pi/2 + pi*mirrored} 0 0"/>
+      <axis xyz="0 0 1"/>
     </joint>
   </xacro:macro>
   <!-- ─── Steering wheel macro (bánh trước lái) ────────────────── -->
-  <!-- Cấu trúc: base_link → steer_joint (revolute,z) → steer_link
-                            → wheel_joint (continuous,y) → wheel    -->
-  <xacro:macro name="steering_wheel" params="name x y">
-    <!-- Link trung gian tại tâm bánh, chỉ mang inertia tối thiểu -->
+  <!-- Cấu trúc (theo repo bạn bè):                                    -->
+  <!--   base_link → steer_joint (revolute, axis Z) → steer_link       -->
+  <!--            → wheel_joint (continuous, axis Z, frame xoay) → wheel-->
+  <!-- steer_link đặt tại mặt phẳng base_link (z=0); bánh hạ xuống      -->
+  <!-- z=wheel_radius-base_link_z. Trục kingpin lái là Z thẳng đứng.    -->
+  <xacro:macro name="steering_wheel" params="name y mirrored">
+    <!-- Link trung gian (kingpin), chỉ mang inertia tối thiểu -->
     <link name="${name}_steer_link">
       <xacro:inertial_box mass="0.001" l="0.01" w="0.01" h="0.01"/>
@@ -88,10 +94,10 @@
       <parent link="base_link"/>
       <child  link="${name}_steer_link"/>
-      <origin xyz="${x} ${y} ${wheel_radius - base_link_z}" rpy="0 0 0"/>
+      <origin xyz="${wheelbase/2} ${y} 0" rpy="0 0 0"/>
       <axis xyz="0 0 1"/>
       <limit lower="-0.5236" upper="0.5236" effort="10.0" velocity="1.0"/>
       <dynamics damping="0.1" friction="0.1"/>
     </joint>
-    <!-- Bánh trước: xoay quanh Y, parent là steer_link -->
+    <!-- Bánh trước: trục quay Z (frame xoay ±90° quanh X), parent là steer_link -->
     <link name="${name}_wheel">
       <visual>
@@ -99,5 +105,4 @@
           <cylinder radius="${wheel_radius}" length="${wheel_width}"/>
         </geometry>
-        <origin xyz="0 0 0" rpy="${pi/2} 0 0"/>
         <material name="black"/>
       </visual>
@@ -106,5 +111,4 @@
           <cylinder radius="${wheel_radius}" length="${wheel_width}"/>
         </geometry>
-        <origin xyz="0 0 0" rpy="${pi/2} 0 0"/>
       </collision>
       <xacro:inertial_cylinder mass="0.15" r="${wheel_radius}" h="${wheel_width}"/>
@@ -113,14 +117,15 @@
       <parent link="${name}_steer_link"/>
       <child  link="${name}_wheel"/>
-      <origin xyz="0 0 0" rpy="0 0 0"/>
-      <axis xyz="0 1 0"/>
+      <origin xyz="0 0 ${wheel_radius - base_link_z}"
+              rpy="${-pi/2 + pi*mirrored} 0 0"/>
+      <axis xyz="0 0 1"/>
     </joint>
   </xacro:macro>
   <!-- Bánh sau dẫn động (JGB37-520) -->
-  <xacro:wheel name="rear_left"   x="${-wheelbase/2}" y="${track_width/2}"/>
-  <xacro:wheel name="rear_right"  x="${-wheelbase/2}" y="${-track_width/2}"/>
+  <xacro:wheel name="rear_left"   y="${track_width/2}"  mirrored="0"/>
+  <xacro:wheel name="rear_right"  y="${-track_width/2}" mirrored="0"/>
   <!-- Bánh trước lái (HTS-20H) — có revolute steer_joint cho Ackermann controller -->
-  <xacro:steering_wheel name="front_left"  x="${wheelbase/2}"  y="${track_width/2}"/>
-  <xacro:steering_wheel name="front_right" x="${wheelbase/2}"  y="${-track_width/2}"/>
+  <xacro:steering_wheel name="front_left"  y="${track_width/2}"  mirrored="0"/>
+  <xacro:steering_wheel name="front_right" y="${-track_width/2}" mirrored="1"/>
   <!-- ─── Gazebo: friction cho bánh ────────────────────────────── -->
   <!-- mu1 = hệ số ma sát tĩnh, mu2 = hệ số ma sát trượt -->
