Commit message: fix(amr_description): cập nhật vị trí camera khớp lắp đặt thật (webcam USB)
IMX-219 chưa về hàng, tạm dùng webcam USB gắn ngang mặt trước xe. Đo thực
tế: cao 10.5cm so với mặt đất, nhô ra phía trước mép chassis 5cm, đặt
ngang (pitch=0) — thay cho vị trí đặt giữ chỗ ban đầu (nghiêng 0.3 rad).

Co-Authored-By: Claude Sonnet 5 <noreply@anthropic.com>

File: src/amr_description/urdf/camera.xacro (robot description, xacro)
@@ -1,6 +1,10 @@
 <?xml version="1.0"?>
 <robot xmlns:xacro="http://www.ros.org/wiki/xacro">
-  <!-- ─── Camera frame (IMX-219 CSI) ───────────────────────────── -->
-  <!-- CẦN ĐIỀU CHỈNH vị trí gắn camera IMX-219 -->
+  <!-- ─── Camera frame ─────────────────────────────────────────── -->
+  <!-- Tạm dùng webcam USB thay IMX-219 (chưa về hàng), gắn ngang mặt
+       trước xe. Đo thực tế (2026-07-03): cao 10.5cm so với mặt đất,
+       nhô ra phía trước 5cm so với mép trước chassis, đặt ngang (pitch=0).
+       base_link_z=0.053m (xem amr_core.xacro) -> z tương đối = 0.105-0.053=0.052m
+       base_length/2=0.1485m -> x tương đối = 0.1485+0.05=0.1985m -->
   <link name="camera_frame">
     <visual>
@@ -14,6 +18,5 @@
     <parent link="base_link"/>
     <child  link="camera_frame"/>
-    <!-- camera thường gắn phía trước, hướng xuống hoặc thẳng -->
-    <origin xyz="0.12 0 0.05" rpy="0 0.3 0"/>
+    <origin xyz="0.1985 0 0.052" rpy="0 0 0"/>
   </joint>
   <!-- Frame optical (ROS convention: z-forward, x-right, y-down) -->

Commit message: fix(firmware): thêm watchdog $VEL timeout - CRITICAL safety, chưa build/nạp
Phát hiện khi test lane_follow_node thật: kill hết node ROS trên Jetson +
gửi cmd_vel=0 nhưng xe vẫn chạy mãi, chỉ dừng khi rút cáp USB STM32. Nguyên
nhân: watchdog nội bộ Hiwonder Motor Driver (tự dừng nếu >2s không nhận
I2C) bị vô hiệu hóa vì STM32 đọc encoder mỗi 10ms bất kể có $VEL mới hay
không -> watchdog phần cứng không bao giờ kích hoạt.

Fix: thêm watchdog riêng ở main.c - track last_vel_rx_ms trong on_cmd_vel(),
nếu quá VEL_WATCHDOG_TIMEOUT_MS (300ms) không nhận $VEL mới thì STM32 tự
gọi DRV_Motor_SetSpeed(0,0). CHƯA build/nạp lên STM32 thật - cần làm ở máy
Windows (STM32CubeIDE) rồi verify: xe tự dừng ~300ms khi mất kết nối Jetson.

feat(amr_perception): thêm lane_follow_node.py (P controller), fix lost-lane
detection (lane_detection_node chỉ publish khi thực sự thấy vạch, tránh xe
chạy mù quáng khi mất dấu). Cập nhật vị trí camera lần 2 (22.5cm/-1.5cm/~7.5°)
sau khi phát hiện làn 46cm rộng hơn FOV camera nằm ngang ban đầu.

Co-Authored-By: Claude Sonnet 5 <noreply@anthropic.com>

File: src/amr_description/urdf/camera.xacro (robot description, xacro)
@@ -2,9 +2,12 @@
 <robot xmlns:xacro="http://www.ros.org/wiki/xacro">
   <!-- ─── Camera frame ─────────────────────────────────────────── -->
-  <!-- Tạm dùng webcam USB thay IMX-219 (chưa về hàng), gắn ngang mặt
-       trước xe. Đo thực tế (2026-07-03): cao 10.5cm so với mặt đất,
-       nhô ra phía trước 5cm so với mép trước chassis, đặt ngang (pitch=0).
-       base_link_z=0.053m (xem amr_core.xacro) -> z tương đối = 0.105-0.053=0.052m
-       base_length/2=0.1485m -> x tương đối = 0.1485+0.05=0.1985m -->
+  <!-- Tạm dùng webcam USB thay IMX-219 (chưa về hàng). Đo thực tế lần 2
+       (2026-07-03, sau khi chỉnh lại để 2 mép vạch làn lọt khung hình):
+       cao 22.5cm so với mặt đất, LÙI VÀO 1.5cm so với mép trước chassis
+       (khác lần đầu: lúc đó nhô ra 5cm, cao 10.5cm, nằm ngang).
+       Nghiêng xuống ~7.5° (ƯỚC LƯỢNG, không chắc chắn — đo bằng mắt,
+       CẦN đo lại chính xác hơn nếu cần TF chuẩn).
+       base_link_z=0.053m (xem amr_core.xacro) -> z tương đối = 0.225-0.053=0.172m
+       base_length/2=0.1485m -> x tương đối = 0.1485-0.015=0.1335m -->
   <link name="camera_frame">
     <visual>
@@ -18,5 +21,5 @@
     <parent link="base_link"/>
     <child  link="camera_frame"/>
-    <origin xyz="0.1985 0 0.052" rpy="0 0 0"/>
+    <origin xyz="0.1335 0 0.172" rpy="0 0.1309 0"/>
   </joint>
   <!-- Frame optical (ROS convention: z-forward, x-right, y-down) -->
